Commit message: Created Simulator class that creates two seperate simulations for the robot. One is for forward and inverse kinematics, the other is for rendering the robot visually for debugging. Created a leg trajectory generator and a leg cycle manager for commanding the legs of the robot. Running the main of the Trajectory Executor class will make the robot walk in simulation. The urdf was also updated

File: Phantom/urdf/Phantom.urdf (robot description, URDF)
Before this commit: robot Phantom, 17 links, 16 joints
Joints:
- joint BL_Motor_1: limit lower= -2 upper=2 effort=1.67 velocity=6.28 -> lower=-1.57 upper=1.57 effort=1.6 velocity=6.55
- joint BL_Motor_2: limit lower= -1.57 upper=1.57 effort=1.67 velocity=6.28 -> lower=-1.57 upper=1.57 effort=1.6 velocity=6.55
- joint BL_Motor_3: limit lower= -1 upper=1 effort=1.67 velocity=6.28 -> lower=-1 upper=1 effort=1.6 velocity=6.55
- joint BR_Motor_1: limit lower= -2 upper=2 effort=1.67 velocity=6.28 -> lower=-1.57 upper=1.57 effort=1.6 velocity=6.55
- joint BR_Motor_2: limit lower= -1.57 upper=1.57 effort=1.67 velocity=6.28 -> lower=-1.57 upper=1.57 effort=1.6 velocity=6.55
- joint BR_Motor_3: limit lower= -1 upper=1 effort=1.67 velocity=6.28 -> lower=-1 upper=1 effort=1.6 velocity=6.55
- joint FL_Motor_1: limit lower= -2 upper=2 effort=1.67 velocity=6.28 -> lower=-1.57 upper=1.57 effort=1.6 velocity=6.55
- joint FL_Motor_2: limit lower= -1.57 upper=1.57 effort=1.67 velocity=6.28 -> lower=-1.57 upper=1.57 effort=1.6 velocity=6.55
- joint FL_Motor_3: limit lower= -1 upper=1 effort=1.67 velocity=6.28 -> lower=-1 upper=1 effort=1.6 velocity=6.55
- joint FR_Motor_1: limit lower= -2 upper=2 effort=1.67 velocity=6.28 -> lower=-1.57 upper=1.57 effort=1.6 velocity=6.55
- joint FR_Motor_2: limit lower= -1.57 upper=1.57 effort=1.67 velocity=6.28 -> lower=-1.57 upper=1.57 effort=1.6 velocity=6.55
- joint FR_Motor_3: limit lower= -1 upper=1 effort=1.67 velocity=6.28 -> lower=-1 upper=1 effort=1.6 velocity=6.55

File: Phantom/urdf/Phantom_connor_edits.urdf (robot description, URDF)
Before this commit: robot Phantom, 17 links, 16 joints
Joints:
- joint BR_Motor_1: origin xyz=-0.06 0.106 0.0396 rpy=3.1416 -1.5708 0 -> xyz=-0.06 0.106 0.0396 rpy=0 -1.5708 0
- joint FL_Motor_1: origin xyz=0.06 -0.106 0.0396 rpy=0 -1.5708 0 -> xyz=0.06 -0.106 0.0396 rpy=3.14159 -1.5708 0
